Commit message: update

File: models/PAPRAS/papras_6dof_2arm_table/papras_6dof_2arm_table.urdf (robot description, URDF)
Before this commit: robot papras_6dof_2arm_table, 34 links, 33 joints
Links:
- link env: geometry collision mesh filename=assets/scene/table_simple.stl; visual mesh filename=assets/scene/table_simple.stl

File: models/PAPRAS/papras_7dof/papras_7dof.urdf (robot description, URDF)
Before this commit: robot papras_7dof, 20 links, 19 joints
Joints:
- joint robot1/wrist_joint: origin xyz=0.006 0.0 0.0 rpy=0 0 0 -> xyz=0.006 0.0 0.0 rpy=1.57 0 0

File: models/PAPRAS/papras_7dof_2arm_table/papras_7dof_2arm_table.urdf (robot description, URDF)
Before this commit: robot papras_7dof_2arm_table, 38 links, 37 joints
Links:
- link env: geometry collision mesh filename=assets/scene/table_simple.stl; visual mesh filename=assets/scene/table_simple.stl
Joints:
- joint robot3/wrist_joint: origin xyz=0.006 0.0 0.0 rpy=0 0 0 -> xyz=0.006 0.0 0.0 rpy=1.57 0 0
- joint robot4/wrist_joint: origin xyz=0.006 0.0 0.0 rpy=0 0 0 -> xyz=0.006 0.0 0.0 rpy=1.57 0 0

File: models/PAPRAS/papras_teleop_bag/papras_teleop_bag.urdf (robot description, URDF)
Before this commit: robot teleop_bag, 36 links, 35 joints
Links:
- added link robot3/rgb_cam_link
- added link robot4/rgb_cam_link
Joints:
- added joint robot3/rgb_cam_mount: type fixed, parent robot3/camera_mount, child robot3/rgb_cam_link, origin xyz=0.0272 -0.049 -0.044 rpy=-0.44505895925855404 0 0
- added joint robot4/rgb_cam_mount: type fixed, parent robot4/camera_mount, child robot4/rgb_cam_link, origin xyz=0.0272 -0.049 -0.044 rpy=-0.44505895925855404 0 0

File: models/humanoids/unitree_g1/g1_29dof.urdf (robot description, URDF)
Before this commit: robot g1_29dof, 40 links, 39 joints
Links:
- added link left_end_effector_link
- added link right_end_effector_link
Joints:
- added joint left_eef_joint: type fixed, parent left_wrist_yaw_link, child left_end_effector_link, origin xyz=0.0415 0.003 0 rpy=-1.57 0 0
- added joint right_eef_joint: type fixed, parent right_wrist_yaw_link, child right_end_effector_link, origin xyz=0.0415 0.003 0 rpy=1.57 0 0
- joint waist_pitch_joint: type fixed -> revolute
- joint waist_roll_joint: type fixed -> revolute
- joint waist_yaw_joint: type fixed -> revolute
