Commit message: modify for ai_worker and vive tracker

File: models/ai_worker/ffw_bg2_follower_without_gripper.urdf (robot description, URDF)
Before this commit: robot ffw_bg2_follower_without_gripper, 23 links, 22 joints
Links:
- link arm_base_link: geometry collision mesh filename=assets/ai_worker/common/follower/body_arm_assy.stl scale=0.001 0.001 0.001; visual mesh filename=assets/ai_worker/common/follower/body_arm_assy.stl scale=0.001 0.001 0.001
- link arm_l_link1: geometry collision mesh filename=assets/ai_worker/common/follower/arm_l_link1.stl scale=0.001 0.001 0.001; visual mesh filename=assets/ai_worker/common/follower/arm_l_link1.stl scale=0.001 0.001 0.001
- link arm_l_link2: geometry collision mesh filename=assets/ai_worker/common/follower/arm_l_link2.stl scale=0.001 0.001 0.001; visual mesh filename=assets/ai_worker/common/follower/arm_l_link2.stl scale=0.001 0.001 0.001
- link arm_l_link3: geometry collision mesh filename=assets/ai_worker/common/follower/arm_l_link3.stl scale=0.001 0.001 0.001; visual mesh filename=assets/ai_worker/common/follower/arm_l_link3.stl scale=0.001 0.001 0.001
- link arm_l_link4: geometry collision mesh filename=assets/ai_worker/common/follower/arm_l_link4.stl scale=0.001 0.001 0.001; visual mesh filename=assets/ai_worker/common/follower/arm_l_link4.stl scale=0.001 0.001 0.001
- link arm_l_link5: geometry collision mesh filename=assets/ai_worker/common/follower/arm_l_link5.stl scale=0.001 0.001 0.001; visual mesh filename=assets/ai_worker/common/follower/arm_l_link5.stl scale=0.001 0.001 0.001
- link arm_l_link6: geometry collision mesh filename=assets/ai_worker/common/follower/arm_l_link6.stl scale=0.001 0.001 0.001; visual mesh filename=assets/ai_worker/common/follower/arm_l_link6.stl scale=0.001 0.001 0.001
- link arm_l_link7: geometry collision mesh filename=assets/ai_worker/common/follower/arm_l_link7.stl scale=0.001 0.001 0.001; visual mesh filename=assets/ai_worker/common/follower/arm_l_link7.stl scale=0.001 0.001 0.001
- link arm_r_link1: geometry collision mesh filename=assets/ai_worker/common/follower/arm_r_link1.stl scale=0.001 0.001 0.001; visual mesh filename=assets/ai_worker/common/follower/arm_r_link1.stl scale=0.001 0.001 0.001
- link arm_r_link2: geometry collision mesh filename=assets/ai_worker/common/follower/arm_r_link2.stl scale=0.001 0.001 0.001; visual mesh filename=assets/ai_worker/common/follower/arm_r_link2.stl scale=0.001 0.001 0.001
- link arm_r_link3: geometry collision mesh filename=assets/ai_worker/common/follower/arm_r_link3.stl scale=0.001 0.001 0.001; visual mesh filename=assets/ai_worker/common/follower/arm_r_link3.stl scale=0.001 0.001 0.001
- link arm_r_link4: geometry collision mesh filename=assets/ai_worker/common/follower/arm_r_link4.stl scale=0.001 0.001 0.001; visual mesh filename=assets/ai_worker/common/follower/arm_r_link4.stl scale=0.001 0.001 0.001
- link arm_r_link5: geometry collision mesh filename=assets/ai_worker/common/follower/arm_r_link5.stl scale=0.001 0.001 0.001; visual mesh filename=assets/ai_worker/common/follower/arm_r_link5.stl scale=0.001 0.001 0.001
- link arm_r_link6: geometry collision mesh filename=assets/ai_worker/common/follower/arm_r_link6.stl scale=0.001 0.001 0.001; visual mesh filename=assets/ai_worker/common/follower/arm_r_link6.stl scale=0.001 0.001 0.001
- link arm_r_link7: geometry collision mesh filename=assets/ai_worker/common/follower/arm_r_link7.stl scale=0.001 0.001 0.001; visual mesh filename=assets/ai_worker/common/follower/arm_r_link7.stl scale=0.001 0.001 0.001
- link base_link: geometry collision mesh filename=assets/ai_worker/ffw_bg2_rev4_follower/base_mobile_assy.stl scale=0.001 0.001 0.001; visual mesh filename=assets/ai_worker/ffw_bg2_rev4_follower/base_mobile_assy.stl scale=0.001 0.001 0.001
- link camera_l_link: geometry collision box size=0.023 0.042 0.042; visual mesh filename=assets/ai_worker/common/follower/d405.stl scale=0.001 0.001 0.001
- link camera_r_link: geometry collision box size=0.023 0.042 0.042; visual mesh filename=assets/ai_worker/common/follower/d405.stl scale=0.001 0.001 0.001
- link head_link1: geometry collision mesh filename=assets/ai_worker/common/follower/head_link1.stl scale=0.001 0.001 0.001; visual mesh filename=assets/ai_worker/common/follower/head_link1.stl scale=0.001 0.001 0.001
- link head_link2: geometry collision mesh filename=assets/ai_worker/common/follower/head_link2.stl scale=0.001 0.001 0.001; visual mesh filename=assets/ai_worker/common/follower/head_link2.stl scale=0.001 0.001 0.001
